Commit message: feat(hw2): add front sonar sectors

File: nsysu_drone_description/urdf/nsysu_drone.urdf (robot description, URDF)
Before this commit: robot nsysu_drone, 5 links, 4 joints
Links:
- added link front_sonar_center_link
- added link front_sonar_left_link
- added link front_sonar_right_link
Joints:
- added joint front_sonar_center_joint: type fixed, parent base_link, child front_sonar_center_link, origin xyz=0.25 0 0 rpy=0 0 0
- added joint front_sonar_left_joint: type fixed, parent base_link, child front_sonar_left_link, origin xyz=0.25 0 0 rpy=0 0 0.436332313
- added joint front_sonar_right_joint: type fixed, parent base_link, child front_sonar_right_link, origin xyz=0.25 0 0 rpy=0 0 -0.436332313

File: nsysu_drone_description/urdf/nsysu_drone.urdf.xacro (robot description, xacro)
@@ -42,4 +42,23 @@
   </joint>
   <link name="sonar_link"/>
+  <!-- Forward sonar sector sensors for Task D obstacle avoidance. -->
+  <joint name="front_sonar_center_joint" type="fixed">
+    <origin rpy="0 0 0" xyz="0.25 0 0"/>
+    <parent link="base_link" />
+    <child link="front_sonar_center_link" />
+  </joint>
+  <link name="front_sonar_center_link"/>
+  <joint name="front_sonar_left_joint" type="fixed">
+    <origin rpy="0 0 ${M_PI/7.2}" xyz="0.25 0 0"/>
+    <parent link="base_link" />
+    <child link="front_sonar_left_link" />
+  </joint>
+  <link name="front_sonar_left_link"/>
+  <joint name="front_sonar_right_joint" type="fixed">
+    <origin rpy="0 0 ${-1 * M_PI/7.2}" xyz="0.25 0 0"/>
+    <parent link="base_link" />
+    <child link="front_sonar_right_link" />
+  </joint>
+  <link name="front_sonar_right_link"/>
   <joint name="front_cam_joint" type="fixed">
     <origin rpy="0 0 0" xyz="0.2 0 0"/>
@@ -170,4 +189,50 @@
     </sensor>
   </gazebo>
+  <xacro:macro name="front_sonar_sensor" params="sensor_name link_name">
+    <gazebo reference="${link_name}">
+      <sensor name="${sensor_name}" type="ray">
+        <always_on>1</always_on>
+        <visualize>1</visualize>
+        <update_rate>30</update_rate>
+        <ray>
+          <scan>
+            <horizontal>
+              <samples>5</samples>
+              <resolution>1.000000</resolution>
+              <min_angle>-0.12</min_angle>
+              <max_angle>0.12</max_angle>
+            </horizontal>
+            <vertical>
+              <samples>5</samples>
+              <resolution>1.000000</resolution>
+              <min_angle>-0.12</min_angle>
+              <max_angle>0.12</max_angle>
+            </vertical>
+          </scan>
+          <range>
+            <min>0.02</min>
+            <max>10</max>
+            <resolution>0.01</resolution>
+          </range>
+          <noise>
+            <type>gaussian</type>
+            <mean>0.0</mean>
+            <stddev>0.01</stddev>
+          </noise>
+        </ray>
+        <plugin name="${sensor_name}" filename="libgazebo_ros_ray_sensor.so">
+          <ros>
+            <namespace>${mp['namespace']}</namespace>
+          </ros>
+          <frame_name>${mp['namespace']}/${link_name}</frame_name>
+          <output_type>sensor_msgs/Range</output_type>
+          <radiation_type>ultrasound</radiation_type>
+        </plugin>
+      </sensor>
+    </gazebo>
+  </xacro:macro>
+  <xacro:front_sonar_sensor sensor_name="front_sonar_center" link_name="front_sonar_center_link"/>
+  <xacro:front_sonar_sensor sensor_name="front_sonar_left" link_name="front_sonar_left_link"/>
+  <xacro:front_sonar_sensor sensor_name="front_sonar_right" link_name="front_sonar_right_link"/>
   <gazebo reference="front_cam_link">
     <sensor name="front_camera" type="camera">

Commit message: feat(hw2): add vertical front sonar sectors

File: nsysu_drone_description/urdf/nsysu_drone.urdf (robot description, URDF)
Before this commit: robot nsysu_drone, 8 links, 7 joints
Links:
- added link front_sonar_down_link
- added link front_sonar_up_link
Joints:
- added joint front_sonar_down_joint: type fixed, parent base_link, child front_sonar_down_link, origin xyz=0.25 0 0 rpy=0 0.261799388 0
- added joint front_sonar_up_joint: type fixed, parent base_link, child front_sonar_up_link, origin xyz=0.25 0 0 rpy=0 -0.261799388 0

File: nsysu_drone_description/urdf/nsysu_drone.urdf.xacro (robot description, xacro)
@@ -61,4 +61,16 @@
   </joint>
   <link name="front_sonar_right_link"/>
+  <joint name="front_sonar_up_joint" type="fixed">
+    <origin rpy="0 ${-1 * M_PI/12} 0" xyz="0.25 0 0"/>
+    <parent link="base_link" />
+    <child link="front_sonar_up_link" />
+  </joint>
+  <link name="front_sonar_up_link"/>
+  <joint name="front_sonar_down_joint" type="fixed">
+    <origin rpy="0 ${M_PI/12} 0" xyz="0.25 0 0"/>
+    <parent link="base_link" />
+    <child link="front_sonar_down_link" />
+  </joint>
+  <link name="front_sonar_down_link"/>
   <joint name="front_cam_joint" type="fixed">
     <origin rpy="0 0 0" xyz="0.2 0 0"/>
@@ -235,4 +247,6 @@
   <xacro:front_sonar_sensor sensor_name="front_sonar_left" link_name="front_sonar_left_link"/>
   <xacro:front_sonar_sensor sensor_name="front_sonar_right" link_name="front_sonar_right_link"/>
+  <xacro:front_sonar_sensor sensor_name="front_sonar_up" link_name="front_sonar_up_link"/>
+  <xacro:front_sonar_sensor sensor_name="front_sonar_down" link_name="front_sonar_down_link"/>
   <gazebo reference="front_cam_link">
     <sensor name="front_camera" type="camera">

Commit message: feat(sonar): add left and right side sonar sensors

File: nsysu_drone_description/urdf/nsysu_drone.urdf (robot description, URDF)
Before this commit: robot nsysu_drone, 10 links, 9 joints
Links:
- added link side_sonar_left_link
- added link side_sonar_right_link
Joints:
- added joint side_sonar_left_joint: type fixed, parent base_link, child side_sonar_left_link, origin xyz=0 0.25 0 rpy=0 0 1.570796326795
- added joint side_sonar_right_joint: type fixed, parent base_link, child side_sonar_right_link, origin xyz=0 -0.25 0 rpy=0 0 -1.570796326795

File: nsysu_drone_description/urdf/nsysu_drone.urdf.xacro (robot description, xacro)
@@ -73,4 +73,16 @@
   </joint>
   <link name="front_sonar_down_link"/>
+  <joint name="side_sonar_left_joint" type="fixed">
+    <origin rpy="0 0 ${M_PI/2}" xyz="0 0.25 0"/>
+    <parent link="base_link" />
+    <child link="side_sonar_left_link" />
+  </joint>
+  <link name="side_sonar_left_link"/>
+  <joint name="side_sonar_right_joint" type="fixed">
+    <origin rpy="0 0 ${-1 * M_PI/2}" xyz="0 -0.25 0"/>
+    <parent link="base_link" />
+    <child link="side_sonar_right_link" />
+  </joint>
+  <link name="side_sonar_right_link"/>
   <joint name="front_cam_joint" type="fixed">
     <origin rpy="0 0 0" xyz="0.2 0 0"/>
@@ -249,4 +261,6 @@
   <xacro:front_sonar_sensor sensor_name="front_sonar_up" link_name="front_sonar_up_link"/>
   <xacro:front_sonar_sensor sensor_name="front_sonar_down" link_name="front_sonar_down_link"/>
+  <xacro:front_sonar_sensor sensor_name="side_sonar_left" link_name="side_sonar_left_link"/>
+  <xacro:front_sonar_sensor sensor_name="side_sonar_right" link_name="side_sonar_right_link"/>
   <gazebo reference="front_cam_link">
     <sensor name="front_camera" type="camera">
